File: PCBv1.kicad_pcb (KiCad board)
At the start: 2 copper layers, 309.6 x 101.6 mm, 156 parts, among them J1 AVR-ISP-6, SW1 `~, SW10 #8, SW11 #9, SW12 #0, SW13 -_, SW14 =+, SW15 BSPC, SW16 PAUSE, SW17 TAB, SW18 Q, SW19 W, SW2 SW_Push_Reset, SW20 E, SW21 R, SW22 T, SW23 Y, SW24 U, SW25 I, SW26 O, SW27 P, SW28 [{, SW29 ]}, SW3 #1, SW30 \|, SW31 NEXT, SW32 CPSLCK, SW33 A, SW34 S, SW35 D, SW36 F, SW37 G, SW38 H, SW39 J, SW4 #2, SW40 K, SW41 L, SW42 ;:, SW43 '", SW44 ENTR, SW45 PRVS, SW46 SHFT, SW47 Z, SW48 X, SW49 C, SW5 #3, SW50 V, SW51 B, SW52 N, SW53 M, SW54 ,<, SW55 .>, SW56 /?, SW57 SHFT, SW58 UP, SW59 DEL, SW6 #4, SW60 CTRL, SW61 WIN, SW62 ALT, SW63 SPC, SW64 ALT, SW65 FN, SW66 CTRL, SW67 LEFT, SW68 DOWN, SW69 RIGHT, SW7 #5, SW8 #6, SW9 #7, U1 ATmega32U4-A, Y1 16MHz

Commit message: locked in
Parts:
- removed D1: PRTR5V0U2X, Package_TO_SOT_SMD:SOT-143
- removed F1: 500m, Fuse:Fuse_1206_3216Metric_Pad1.42x1.75mm_HandSolder
- removed R6, R7: 22, Resistor_SMD:R_0805_2012Metric_Pad1.20x1.40mm_HandSolder
- removed R8, R9: 5.1k, Resistor_SMD:R_0805_2012Metric_Pad1.20x1.40mm_HandSolder
- removed USB1: HRO-TYPE-C-31-M-12, Type-C:HRO-TYPE-C-31-M-12-HandSoldering
- added J2: Conn_01x04_MountingPin, Connector_JST:JST_SH_SM04B-SRSS-TB_1x04-1MP_P1.00mm_Horizontal, B.Cu at (218.8, 67.3)
Connections:
- net Net-(U1-XTAL1) renamed XTAL1
- net Net-(U1-XTAL2) renamed XTAL2
- U1 pad 1: row3 -> unconnected-(U1-PE6-Pad1)
- U1 pad 10: MOSI -> MISO
- U1 pad 11: MISO -> col7
- U1 pad 42: unconnected-(U1-AREF-Pad42) -> row3
- U1 pad 8: col7 -> MOSI
Routing:
- net DP: track 84.6 -> 0.00 mm
- net D+: track 7.20 -> 90.0 mm
- net DN: track 82.6 -> 0.00 mm
- net D-: track 7.20 -> 88.9 mm
- net GND: track 282.7 -> 248.1 mm, vias 12 -> 8
- net VCC: track 24.7 -> 0.00 mm, vias 2 -> 0
- net +5V: track 201.6 -> 219.4 mm
- net Net-(USB1-CC2): track 10.6 -> 0.00 mm
- net Net-(USB1-CC1): track 10.3 -> 0.00 mm
- net row3: track 429.6 -> 421.4 mm, vias 6 -> 4
- net col7: track 97.2 -> 94.4 mm
- net MOSI: track 60.6 -> 58.3 mm
- net SCK: track 61.2 -> 59.0 mm
- net MISO: track 67.6 -> 65.7 mm, vias 5 -> 3
- net row0: track 514.2 -> 513.7 mm
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- added copper zone on B.Cu, net GND

Commit message: done
Other:
- board size 309.6 x 101.6 mm -> 309.6 x 100 mm
Changed lines of the file:
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@@
 		)
-	)
-	(gr_line
-		(start 214.3125 60.325)
-		(end 214.3125 59.53125)
-		(stroke
-			(width 0.05)
-			(type default)
-		)
-		(layer "Edge.Cuts")
 	)
 	(gr_arc
@@
 	)
 	(gr_line
-		(start 373.0625 61.11875)
-		(end 229.39375 61.11875)
+		(start 213.51875 61.11875)
+		(end 227.80625 61.11875)
 		(stroke
 			(width 0.05)
@@
 	)
 	(gr_line
-		(start 227.0125 59.53125)
-		(end 227.0125 60.316091)
+		(start 373.0625 61.11875)
+		(end 229.39375 61.11875)
 		(stroke
 			(width 0.05)
@@
 		(mid 66.578702 61.816202)
 		(end 68.2625 61.11875)
-		(stroke
-			(width 0.05)
-			(type default)
-		)
-		(layer "Edge.Cuts")
-	)
-	(gr_arc
-		(start 214.3125 60.325)
-		(mid 214.080016 60.886266)
-		(end 213.51875 61.11875)
 		(stroke
 			(width 0.05)
@@
 	)
 	(gr_line
-		(start 214.3125 59.53125)
-		(end 227.0125 59.53125)
-		(stroke
-			(width 0.05)
-			(type default)
-		)
-		(layer "Edge.Cuts")
-	)
-	(gr_line
 		(start 227.80625 61.118749)
 		(end 229.39375 61.11875)
@@
 		(stroke
 			(width 0.05)
-			(type default)
-		)
-		(layer "Edge.Cuts")
-	)
-	(gr_arc
-		(start 227.80625 61.11875)
-		(mid 227.244984 60.886266)
-		(end 227.0125 60.325)
-		(stroke
-			(width 0.05)

Commit message: idek
Routing:
- net row3: track 421.4 -> 422.0 mm
- net col12: track 213.9 -> 214.5 mm
- net row2: track 474.2 -> 474.8 mm
