File: PCBv1.kicad_pcb (KiCad board)
At the start: 2 copper layers, 309.6 x 100 mm, 150 parts, among them J1 AVR-ISP-6, J2 Conn_01x04_MountingPin, SW1 `~, SW10 #8, SW11 #9, SW12 #0, SW13 -_, SW14 =+, SW15 BSPC, SW16 PAUSE, SW17 TAB, SW18 Q, SW19 W, SW2 SW_Push_Reset, SW20 E, SW21 R, SW22 T, SW23 Y, SW24 U, SW25 I, SW26 O, SW27 P, SW28 [{, SW29 ]}, SW3 #1, SW30 \|, SW31 NEXT, SW32 CPSLCK, SW33 A, SW34 S, SW35 D, SW36 F, SW37 G, SW38 H, SW39 J, SW4 #2, SW40 K, SW41 L, SW42 ;:, SW43 '", SW44 ENTR, SW45 PRVS, SW46 SHFT, SW47 Z, SW48 X, SW49 C, SW5 #3, SW50 V, SW51 B, SW52 N, SW53 M, SW54 ,<, SW55 .>, SW56 /?, SW57 SHFT, SW58 UP, SW59 DEL, SW6 #4, SW60 CTRL, SW61 WIN, SW62 ALT, SW63 SPC, SW64 ALT, SW65 FN, SW66 CTRL, SW67 LEFT, SW68 DOWN, SW69 RIGHT, SW7 #5, SW8 #6, SW9 #7, U1 ATmega32U4-A, Y1 16MHz

Commit message: fix row3 pin
Connections:
- U1 pad 1: unconnected-(U1-PE6-Pad1) -> row3
- U1 pad 42: row3 -> unconnected-(U1-AREF-Pad42)
Routing:
- net row3: track 422.0 -> 422.7 mm, vias 4 -> 5
Changed lines of the file:
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@@
 	(net 99 "col14")
 	(net 100 "unconnected-(U1-PD0-Pad18)")
-	(net 101 "unconnected-(U1-PB7-Pad12)")
+	(net 101 "unconnected-(U1-AREF-Pad42)")
 	(net 102 "XTAL2")
-	(net 103 "unconnected-(U1-PE6-Pad1)")
+	(net 103 "unconnected-(U1-PB7-Pad12)")
 	(footprint "MX_Only:MXOnly-1.25U-NoLED"
 		(layer "F.Cu")
@@
 			(size 1.5 0.55)
 			(layers "B.Cu" "B.Mask" "B.Paste")
-			(net 103 "unconnected-(U1-PE6-Pad1)")
+			(net 53 "row3")
 			(pinfunction "PE6")
-			(pintype "bidirectional+no_connect")
+			(pintype "bidirectional")
 		)
 		(pad "2" smd rect
@@
 			(size 1.5 0.55)
 			(layers "B.Cu" "B.Mask" "B.Paste")
-			(net 101 "unconnected-(U1-PB7-Pad12)")
+			(net 103 "unconnected-(U1-PB7-Pad12)")
 			(pinfunction "PB7")
 			(pintype "bidirectional+no_connect")
@@
 			(size 1.5 0.55)
 			(layers "B.Cu" "B.Mask" "B.Paste")
-			(net 53 "row3")
+			(net 101 "unconnected-(U1-AREF-Pad42)")
 			(pinfunction "AREF")
-			(pintype "passive")
+			(pintype "passive+no_connect")
 		)
 		(pad "43" smd rect
@@
 	)
 	(segment
+		(start 215 143.5)
+		(end 215.5 143.5)
+		(width 0.2)
+		(layer "F.Cu")
+		(net 53)
+	)
+	(segment
 		(start 204.47 137.16)
 		(end 202.693 137.16)
@@
 		(net 53)
 	)
+	(segment
+		(start 212.5 144)
+		(end 214.5 144)
+		(width 0.2)
+		(layer "F.Cu")
+		(net 53)
+	)
+	(segment
+		(start 214.5 144)
+		(end 215 143.5)
+		(width 0.2)
+		(layer "F.Cu")
+		(net 53)
+	)
 	(via
 		(at 202.693 137.16)
@@
 	)
 	(via
+		(at 212.5 144)
+		(size 0.6)
+		(drill 0.3)
+		(layers "F.Cu" "B.Cu")
+		(net 53)
+	)
+	(via
 		(at 204.47 137.16)
 		(size 0.6)
@@
 	)
 	(segment
-		(start 200.682281 141.516)
-		(end 199.286281 142.912)
+		(start 145.885 141.516)
+		(end 84.112 141.516)
 		(width 0.2)
 		(layer "B.Cu")
@@
 	)
 	(segment
-		(start 83.66125 141.06525)
-		(end 83.66125 136.525)
+		(start 150.495 139.319)
+		(end 148.082 139.319)
 		(width 0.2)
 		(layer "B.Cu")
@@
 	)
 	(segment
-		(start 84.112 141.516)
-		(end 83.66125 141.06525)
+		(start 285.4325 137.16)
+		(end 267.6525 137.16)
 		(width 0.2)
 		(layer "B.Cu")
@@
 	)
 	(segment
-		(start 285.4325 137.16)
-		(end 267.6525 137.16)
+		(start 113.9825 137.16)
+		(end 104.147095 137.16)
 		(width 0.2)
 		(layer "B.Cu")
@@
 	)
 	(segment
-		(start 113.9825 137.16)
-		(end 104.147095 137.16)
+		(start 148.082 139.319)
+		(end 145.885 141.516)
+		(width 0.2)
+		(layer "B.Cu")
+		(net 53)
+	)
+	(segment
+		(start 212.5 144)
+		(end 205.705813 144)
 		(width 0.2)
 		(layer "B.Cu")
@@
 	)
 	(segment
+		(start 84.112 141.516)
+		(end 83.66125 141.06525)
+		(width 0.2)
+		(layer "B.Cu")
+		(net 53)
+	)
+	(segment
 		(start 286.7025 137.16)
 		(end 286.0675 136.525)
@@
 	)
 	(segment
-		(start 150.495 139.319)
-		(end 148.082 139.319)
+		(start 98.933 137.16)
+		(end 84.29625 137.16)
 		(width 0.2)
 		(layer "B.Cu")
@@
 	)
 	(segment
-		(start 98.933 137.16)
-		(end 84.29625 137.16)
+		(start 200.682281 141.516)
+		(end 199.286281 142.912)
 		(width 0.2)
 		(layer "B.Cu")
@@
 	)
 	(segment
-		(start 203.221813 141.516)
-		(end 200.682281 141.516)
-		(width 0.2)
-		(layer "B.Cu")
-		(net 53)
-	)
-	(segment
 		(start 190.1825 137.16)
 		(end 172.4025 137.16)
@@
 	)
 	(segment
-		(start 145.885 141.516)
-		(end 84.112 141.516)
+		(start 204.47 137.16)
+		(end 209.2325 137.16)
 		(width 0.2)
 		(layer "B.Cu")
@@
 	)
 	(segment
-		(start 204.47 137.16)
-		(end 209.2325 137.16)
+		(start 83.66125 141.06525)
+		(end 83.66125 136.525)
 		(width 0.2)
 		(layer "B.Cu")
@@
 	)
 	(segment
-		(start 208.318313 146.6125)
-		(end 203.221813 141.516)
+		(start 203.221813 141.516)
+		(end 200.682281 141.516)
 		(width 0.2)
 		(layer "B.Cu")
@@
 	)
 	(segment
-		(start 172.4025 137.16)
-		(end 171.7675 136.525)
+		(start 154.088 142.912)
+		(end 150.495 139.319)
 		(width 0.2)
 		(layer "B.Cu")
@@
 	)
 	(segment
-		(start 148.082 139.319)
-		(end 145.885 141.516)
+		(start 172.4025 137.16)
+		(end 171.7675 136.525)
 		(width 0.2)
 		(layer "B.Cu")
@@
 	)
 	(segment
-		(start 152.0825 137.16)
-		(end 134.3025 137.16)
+		(start 199.286281 142.912)
+		(end 154.088 142.912)
 		(width 0.2)
 		(layer "B.Cu")
@@
 	)
 	(segment
-		(start 228.2825 137.16)
-		(end 228.9175 136.525)
+		(start 205.705813 144)
+		(end 203.221813 141.516)
+		(width 0.2)
+		(layer "B.Cu")
+		(net 53)
+	)
+	(segment
+		(start 152.0825 137.16)
+		(end 134.3025 137.16)
 		(width 0.2)
 		(layer "B.Cu")
@@
 	)
 	(segment
-		(start 213.88625 146.6125)
-		(end 208.318313 146.6125)
+		(start 228.2825 137.16)
+		(end 228.9175 136.525)
 		(width 0.2)
 		(layer "B.Cu")
@@
 	)
 	(segment
-		(start 199.286281 142.912)
-		(end 154.088 142.912)
-		(width 0.2)
-		(layer "B.Cu")
-		(net 53)
-	)
-	(segment
 		(start 209.2325 137.16)
 		(end 209.8675 136.525)
@@
 	)
 	(segment
-		(start 154.088 142.912)
-		(end 150.495 139.319)
-		(width 0.2)
-		(layer "B.Cu")
-		(net 53)
-	)
-	(segment
 		(start 202.693 137.16)
 		(end 191.4525 137.16)
@@
 		(net 102)
 	)
+	(segment
+		(start 225.27375 145)
+		(end 225.28625 145.0125)
+		(width 0.2)
+		(layer "B.Cu")
+		(net 103)
+	)
 	(zone

Commit message: idek
Routing:
- net row3: track 422.7 -> 422.9 mm, vias 5 -> 6
Changed lines of the file:
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@@
-	)
-	(segment
-		(start 215 143.5)
-		(end 215.5 143.5)
-		(width 0.2)
-		(layer "F.Cu")
-		(net 53)
 	)
 	(segment
@@
 	)
 	(via
+		(at 215 143.5)
+		(size 0.6)
+		(drill 0.3)
+		(layers "F.Cu" "B.Cu")
+		(net 53)
+	)
+	(via
 		(at 202.693 137.16)
 		(size 0.6)
@@
 		(drill 0.3)
 		(layers "F.Cu" "B.Cu")
+		(net 53)
+	)
+	(segment
+		(start 215 143.5)
+		(end 215.39875 143.5)
+		(width 0.2)
+		(layer "B.Cu")
 		(net 53)
 	)
@@
 		(width 0.2)
 		(layer "B.Cu")
+		(net 53)
+	)
+	(segment
+		(start 215.39875 143.5)
+		(end 215.58625 143.3125)
+		(width 0.2)
+		(layer "B.Cu")
